File: engineering_plane.kicad_pcb (KiCad board)
At the start: 2 copper layers, 100 x 100 mm, 0 parts

Commit message: feat: power section done, onto sensors
Parts:
- added A1: RaspberryPi_Pico_W, Module:RaspberryPi_Pico_W_SMD_HandSolder, F.Cu at (160.9, 89.1)
- added C1: 10u, Capacitor_SMD:C_1206_3216Metric, F.Cu at (186.2, 93.6)
- added C10: 10u, Capacitor_SMD:C_1206_3216Metric, F.Cu at (189.1, 109.2)
- added C11: 0.1u, Capacitor_SMD:C_0805_2012Metric, F.Cu at (188.5, 111.4)
- added C12: 0.1u, Capacitor_SMD:C_0805_2012Metric, F.Cu at (191.3, 116.3)
- added C13: 22u, Capacitor_SMD:C_1206_3216Metric, F.Cu at (188.3, 120.8)
- added C14: 22u, Capacitor_SMD:C_1206_3216Metric, F.Cu at (190.9, 120.8)
- added C15: 100p, Capacitor_SMD:C_0805_2012Metric, F.Cu at (183.8, 116.8)
- added C2: 10u, Capacitor_SMD:C_1206_3216Metric, F.Cu at (186.2, 96.1)
- added C3: 0.1u, Capacitor_SMD:C_0805_2012Metric, F.Cu at (186.2, 91.4)
- added C4: 100u, Capacitor_SMD:CP_Elec_6.3x7.7, F.Cu at (186.4, 100.8)
- added C5: 0.1u, Capacitor_SMD:C_0805_2012Metric, F.Cu at (183.4, 87.4)
- added C6: 22u, Capacitor_SMD:C_1206_3216Metric, F.Cu at (189.8, 80.8)
- added C7: 22u, Capacitor_SMD:C_1206_3216Metric, F.Cu at (192.2, 80.8)
- added C8: 100p, Capacitor_SMD:C_0805_2012Metric, F.Cu at (185.6, 83.3)
- added C9: 10u, Capacitor_SMD:C_1206_3216Metric, F.Cu at (189.1, 106.8)
- added D1: SMF15A, Diode_SMD:D_SMF, F.Cu at (193.0, 101.9)
- added D2: SS24, Diode_SMD:D_SMA, F.Cu at (175.9, 70.3)
- added J1: Conn_01x02_Pin, Connector_AMASS:AMASS_XT30PW-M_1x02_P2.50mm_Horizontal, F.Cu at (196.5, 105.5)
- added L1: 10u, Inductor_SMD:L_7.3x7.3_H4.5, F.Cu at (192.4, 87.3)
- added L2: 10u, Inductor_SMD:L_7.3x7.3_H4.5, F.Cu at (196.8, 116.8)
- added R1: 100k, PCM_SparkFun-Resistor:R_0603_1608Metric, F.Cu at (187.4, 83.4)
- added R2: 13.3k, PCM_SparkFun-Resistor:R_0603_1608Metric, F.Cu at (182.9, 84.1)
- added R3: 100k, PCM_SparkFun-Resistor:R_0603_1608Metric, F.Cu at (185.6, 117.0)
- added R4: 11k, PCM_SparkFun-Resistor:R_0603_1608Metric, F.Cu at (185.5, 113.9)
- added U1: TPS54302DDCR, TPS54302:SOT95P280X110-6N, F.Cu at (186.2, 87.7)
- added U2: TPS54302DDCR, TPS54302:SOT95P280X110-6N, F.Cu at (188.5, 115.1)
Routing:
- net VBATT: track 0.00 -> 38.7 mm
- net GND: track 0.00 -> 32.5 mm, vias 0 -> 30
- net +5V: track 0.00 -> 27.4 mm
- net +6V: track 0.00 -> 17.9 mm
- net Net-(U1-SW): track 0.00 -> 7.78 mm
- net Net-(U2-SW): track 0.00 -> 6.71 mm
- net /5v_div: track 0.00 -> 6.11 mm
- net Net-(A1-VSYS): track 0.00 -> 5.64 mm
- net /6v_div: track 0.00 -> 5.47 mm
- net Net-(U2-BOOT): track 0.00 -> 2.20 mm
- net Net-(U1-BOOT): track 0.00 -> 1.82 mm

Commit message: feat: schematic mostly finished, onto the PCB
Parts:
- added C11: 100n, Capacitor_SMD:C_0603_1608Metric, F.Cu at (137.1, 85.1)
- added C15: 1u, Capacitor_SMD:C_0603_1608Metric, F.Cu at (236.9, 94.7)
- added C16: 1u, Capacitor_SMD:C_0603_1608Metric, F.Cu at (236.9, 92.2)
- added C22: 100n, Capacitor_SMD:C_0603_1608Metric, F.Cu at (231.6, 146.8)
- added C23: 100n, Capacitor_SMD:C_0603_1608Metric, F.Cu at (231.6, 149.4)
- added C24: 1u, Capacitor_SMD:C_0603_1608Metric, F.Cu at (231.6, 151.9)
- added C25: 100n, Capacitor_SMD:C_0603_1608Metric, F.Cu at (243.7, 146.8)
- added C26: 100n, Capacitor_SMD:C_0603_1608Metric, F.Cu at (243.7, 149.4)
- added C27: 1u, Capacitor_SMD:C_0603_1608Metric, F.Cu at (243.7, 151.9)
- added C4: 470u, Capacitor_SMD:CP_Elec_10x10.5, F.Cu at (173.0, 117.9)
- added C7: 10u, Capacitor_SMD:C_1206_3216Metric, F.Cu at (177.3, 124.9)
- added C9: 10u, Capacitor_SMD:C_1206_3216Metric, F.Cu at (177.6, 76.8)
- added D2: SMF6V5A, Diode_SMD:D_SMF, F.Cu at (181.5, 116.3)
- added IC1: LP5907MFX-3.3_NOPB, eng_plane_lib:SOT95P280X145-5M, F.Cu at (255.9, 148.1)
- added IC2: BMI270, eng_plane_lib:BMI270, F.Cu at (236.6, 148.4)
- added IC3: BMP390, eng_plane_lib:BMP390, F.Cu at (248.2, 148.1)
- added J1: Conn_01x01_Pin, Connector_Wire:SolderWire-2sqmm_1x01_D2mm_OD3.9mm, F.Cu at (206.2, 92.8)
- added J10: 171857-0003, eng_plane_lib:1718570003, F.Cu at (180.1, 67.0)
- added J2: Conn_01x01_Pin, Connector_Wire:SolderWire-2sqmm_1x01_D2mm_OD3.9mm, F.Cu at (206.2, 112.7)
- added J3: JST_1mm_4, PCM_SparkFun-Connector:JST_1x04_P1.0mm_Horizontal_SMD, F.Cu at (115.0, 111.5)
- added J4: JST_1mm_4, PCM_SparkFun-Connector:JST_1x04_P1.0mm_Horizontal_SMD, F.Cu at (115.0, 86.9)
- added J6: JST_1mm_4, PCM_SparkFun-Connector:JST_1x04_P1.0mm_Horizontal_SMD, F.Cu at (115.0, 121.0)
- added J7: 171857-0003, eng_plane_lib:1718570003, F.Cu at (185.0, 133.0)
- added J8: 171857-0003, eng_plane_lib:1718570003, F.Cu at (175.0, 133.0)
- added J9: 171857-0003, eng_plane_lib:1718570003, F.Cu at (190.1, 67.0)
- added L3: 600 Ohm, PCM_SparkFun-Capacitor:C_0805_2012Metric, F.Cu at (235.5, 114.8)
- added L4: 600 Ohm, PCM_SparkFun-Capacitor:C_0805_2012Metric, F.Cu at (229.0, 114.8)
- added R11: 100, PCM_SparkFun-Resistor:R_0603_1608Metric, F.Cu at (257.5, 92.2)
- added R12: 100, PCM_SparkFun-Resistor:R_0603_1608Metric, F.Cu at (257.5, 97.2)
- added R13: 100, PCM_SparkFun-Resistor:R_0603_1608Metric, F.Cu at (257.5, 102.2)
- added R14: 100, PCM_SparkFun-Resistor:R_0603_1608Metric, F.Cu at (257.5, 107.2)
- added R15: 10k, PCM_SparkFun-Resistor:R_0603_1608Metric, F.Cu at (257.5, 94.7)
- added R16: 10k, PCM_SparkFun-Resistor:R_0603_1608Metric, F.Cu at (257.5, 99.7)
- added R17: 10k, PCM_SparkFun-Resistor:R_0603_1608Metric, F.Cu at (257.5, 104.7)
- added R18: 10k, PCM_SparkFun-Resistor:R_0603_1608Metric, F.Cu at (257.5, 109.7)
- added R3: 47k, PCM_SparkFun-Resistor:R_0603_1608Metric, F.Cu at (177.7, 100.8)
- added R4: 1k, PCM_SparkFun-Resistor:R_0603_1608Metric, F.Cu at (138.8, 85.1)
- added R5: 100, PCM_SparkFun-Resistor:R_0603_1608Metric, F.Cu at (241.0, 103.0)
- added R6: 100, PCM_SparkFun-Resistor:R_0603_1608Metric, F.Cu at (241.0, 105.6)
- added R7: 100, PCM_SparkFun-Resistor:R_0603_1608Metric, F.Cu at (241.0, 108.1)
- added R8: 100, PCM_SparkFun-Resistor:R_0603_1608Metric, F.Cu at (241.0, 110.6)
- added REF**: MountingHole_3.2mm_M3_Pad, MountingHole:MountingHole_3.2mm_M3_Pad, F.Cu at (205.0, 130.0)
- added REF**: MountingHole_3.2mm_M3_Pad, MountingHole:MountingHole_3.2mm_M3_Pad, F.Cu at (205.0, 70.0)
- added REF**: MountingHole_3.2mm_M3_Pad, MountingHole:MountingHole_3.2mm_M3_Pad, F.Cu at (115.0, 130.0)
- added REF**: MountingHole_3.2mm_M3_Pad, MountingHole:MountingHole_3.2mm_M3_Pad, F.Cu at (115.0, 70.0)
- A1: footprint Module:RaspberryPi_Pico_W_SMD_HandSolder -> Module:RaspberryPi_Pico_Common_SMD
- moved D1 51.7 mm to (126.1, 84.3), turned to 90 degrees
- moved A1 17.1 mm to (147.7, 100.0), turned to 90 degrees
- moved D3 0.53 mm to (193.0, 102.5)
- moved C21 0.12 mm to (183.7, 116.9)
- renumbered C8 to C10, C9 to C12, C10 to C13, C11 to C14, C12 to C17, C13 to C18, C14 to C19, C4 to C20, C15 to C21, C7 to C8, D2 to D1, D1 to D3, J1 to J5, R4 to R10, R3 to R9
Connections:
- A1 pad 36: +3V3 -> unconnected-(A1-3V3-Pad36)
Routing:
- net +6V: track 17.9 -> 66.3 mm
- net +5V: track 27.4 -> 13.1 mm
- net Net-(A1-VSYS): track 5.64 -> 0.00 mm
- net GND: track 32.5 -> 32.0 mm
- added copper zone on F.Cu, net +6V
- added copper zone on F.Cu, net VBATT
- removed copper zone on B.Cu, net GND
Other:
- board outline removed

Commit message: sisyphus goes hard, awaiting review.
Parts:
- added C28: 10u, Capacitor_SMD:C_0603_1608Metric, F.Cu at (115.9, 125.7)
- added C29: 1u, Capacitor_SMD:C_0603_1608Metric, F.Cu at (119.0, 123.8)
- added C30: 1u, Capacitor_SMD:C_0603_1608Metric, F.Cu at (120.5, 123.8)
- added C31: 100n, Capacitor_SMD:C_0603_1608Metric, F.Cu at (113.4, 118.7)
- added IC4: MMC5983MA, eng_plane_lib:MMC5983MA, F.Cu at (115.4, 122.4)
- added J1: JST_1mm_4, PCM_SparkFun-Connector:JST_1x04_P1.0mm_Horizontal_SMD, F.Cu at (116.1, 108.2)
- added J12: Conn_01x07_Pin, Connector_PinHeader_2.54mm:PinHeader_1x07_P2.54mm_Vertical, F.Cu at (127.2, 101.1)
- added J14: Conn_01x04_Pin, Connector_PinHeader_2.54mm:PinHeader_1x04_P2.54mm_Vertical, F.Cu at (126.7, 83.2)
- added J15: Conn_01x03, eng_plane_lib:1718564003, F.Cu at (173.7, 109.9)
- added L5: 600 Ohm, PCM_SparkFun-Capacitor:C_0805_2012Metric, F.Cu at (123.3, 123.1)
- added R1: 4.7k, PCM_SparkFun-Resistor:R_0603_1608Metric, F.Cu at (160.1, 110.4)
- added R2: 4.7k, PCM_SparkFun-Resistor:R_0603_1608Metric, F.Cu at (164.1, 102.8)
- added R21: 4.7k, PCM_SparkFun-Resistor:R_0603_1608Metric, F.Cu at (118.0, 116.4)
- added R22: 4.7k, PCM_SparkFun-Resistor:R_0603_1608Metric, F.Cu at (117.1, 114.5)
- added R23: 100, PCM_SparkFun-Resistor:R_0603_1608Metric, F.Cu at (154.1, 116.3)
- added R24: 10k, PCM_SparkFun-Resistor:R_0603_1608Metric, F.Cu at (156.6, 117.4)
- C10, C14, C17, C3, C5: footprint Capacitor_SMD:C_0805_2012Metric -> Capacitor_SMD:C_0603_1608Metric
- H1, H2, H3, H4: renamed from REF**; value MountingHole_3.2mm_M3_Pad -> MountingHole_Pad
- R6: renamed from R4; value 1k -> 10k
- U1, U2: footprint TPS54302:SOT95P280X110-6N -> eng_plane_lib:SOT95P280X110-6N
- moved R10 118.1 mm to (127.5, 78.0)
- moved R9 118.1 mm to (127.5, 75.5)
- moved R7 114.4 mm to (127.6, 88.3)
- moved R8 114.4 mm to (127.6, 90.8)
- moved R13 107.3 mm to (154.3, 121.3), turned to 180 degrees
- moved R14 106.6 mm to (154.4, 124.0), turned to 180 degrees
- moved R16 104.6 mm to (154.2, 90.8), turned to 180 degrees
- moved R17 104.2 mm to (156.6, 120.4), turned to -90 degrees
- moved R18 103.8 mm to (156.8, 124.7), turned to 90 degrees
- moved R15 103.3 mm to (154.3, 98.6), turned to 180 degrees
- moved R20 102.6 mm to (156.6, 91.5), turned to 90 degrees
- moved IC1 102.3 mm to (171.5, 90.3), turned to -90 degrees
- moved R19 101.0 mm to (156.6, 99.4), turned to 90 degrees
- moved IC3 97.2 mm to (159.9, 107.5)
- moved C25 93.8 mm to (159.9, 104.6)
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- renumbered J9 to J10, J10 to J11, J1 to J2, J2 to J3, J3 to J4, J4 to J5, J5 to J6, J6 to J7, J7 to J8, J8 to J9, R8 to R10, R9 to R11, R10 to R12, R11 to R13, R12 to R14, R13 to R15, R14 to R16, R15 to R17, R16 to R18, R17 to R19, R18 to R20, R1 to R3, R2 to R4, R3 to R5, R5 to R7, R6 to R8, R7 to R9
Connections:
- A1 pad 1: unconnected-(A1-GPIO0-Pad1) -> /rc_rx
- A1 pad 10: unconnected-(A1-GPIO7-Pad10) -> /i2c1_scl
- A1 pad 11: unconnected-(A1-GPIO8-Pad11) -> Net-(A1-GPIO8)
- A1 pad 12: unconnected-(A1-GPIO9-Pad12) -> Net-(A1-GPIO9)
- A1 pad 14: unconnected-(A1-GPIO10-Pad14) -> Net-(A1-GPIO10)
- A1 pad 15: unconnected-(A1-GPIO11-Pad15) -> Net-(A1-GPIO11)
- A1 pad 16: unconnected-(A1-GPIO12-Pad16) -> Net-(A1-GPIO12)
- A1 pad 17: unconnected-(A1-GPIO13-Pad17) -> /mmc_int
- A1 pad 2: unconnected-(A1-GPIO1-Pad2) -> /rc_tx
- A1 pad 21: unconnected-(A1-GPIO16-Pad21) -> /pwm0_a
- A1 pad 22: unconnected-(A1-GPIO17-Pad22) -> /pwm0_b
- A1 pad 24: unconnected-(A1-GPIO18-Pad24) -> /pwm1_a
- A1 pad 25: unconnected-(A1-GPIO19-Pad25) -> /bmp_int
- A1 pad 26: unconnected-(A1-GPIO20-Pad26) -> /i2c0_sda
- A1 pad 27: unconnected-(A1-GPIO21-Pad27) -> /i2c0_scl
- A1 pad 29: unconnected-(A1-GPIO22-Pad29) -> /bmi_int
- A1 pad 31: unconnected-(A1-GPIO26_ADC0-Pad31) -> /pwm5_a
- A1 pad 32: unconnected-(A1-GPIO27_ADC1-Pad32) -> /adc_v
- A1 pad 34: unconnected-(A1-GPIO28_ADC2-Pad34) -> /pwm6_a
- A1 pad 4: unconnected-(A1-GPIO2-Pad4) -> Net-(A1-GPIO2)
- A1 pad 5: unconnected-(A1-GPIO3-Pad5) -> Net-(A1-GPIO3)
- A1 pad 6: unconnected-(A1-GPIO4-Pad6) -> /gps_rx
- A1 pad 7: unconnected-(A1-GPIO5-Pad7) -> /gps_tx
- A1 pad 9: unconnected-(A1-GPIO6-Pad9) -> /i2c1_sda
- C22 pad 2: +3V3 -> /bmi270/filter_3v3
- C23 pad 2: Net-(IC2-VDD) -> /bmi270/filter_3v3
- C24 pad 1: Net-(IC2-VDD) -> /bmi270/filter_3v3
- C25 pad 2: +3V3 -> /bmp390/filter_3v3
- C26 pad 2: Net-(IC3-VDD) -> /bmp390/filter_3v3
- C27 pad 1: Net-(IC3-VDD) -> /bmp390/filter_3v3
- IC2 pad 12: +3V3 -> /bmi270/filter_3v3
- IC2 pad 13: /bmi270/BMI_SCL -> /i2c0_scl
- IC2 pad 14: /bmi270/BMI_SDA -> /i2c0_sda
- IC2 pad 4: /bmi270/BMI_INT1 -> /bmi_int
- IC2 pad 5: +3V3 -> /bmi270/filter_3v3
- IC2 pad 8: Net-(IC2-VDD) -> /bmi270/filter_3v3
- IC3 pad 1: +3V3 -> /bmp390/filter_3v3
- IC3 pad 10: Net-(IC3-VDD) -> /bmp390/filter_3v3
- IC3 pad 2: /bmp390/bmp_SCL -> /i2c0_scl
- IC3 pad 4: /bmp390/bmp_SDA -> /i2c0_sda
- IC3 pad 6: +3V3 -> /bmp390/filter_3v3
- IC3 pad 7: /bmp390/bmp_int -> /bmp_int
- J5 pad 2: /pitot_scl -> /i2c1_scl
- J5 pad 3: /pitot_sda -> /i2c1_sda
- L3 pad 1: Net-(IC2-VDD) -> /bmi270/filter_3v3
- L4 pad 1: Net-(IC3-VDD) -> /bmp390/filter_3v3
- R13 pad 2: /servos/servo_pwm1 -> /pwm0_b
- R14 pad 2: /servos/servo_pwm2 -> /pwm0_a
- R15 pad 2: /servos/servo_pwm3 -> /pwm5_a
- R16 pad 2: /servos/servo_pwm4 -> /pwm6_a
Routing:
- net +3V3: track 0.00 -> 183.2 mm
- net +5V: track 13.1 -> 142.2 mm, vias 0 -> 4
- net Net-(J10-Pad3): track 0.00 -> 45.2 mm, vias 0 -> 1
- net /i2c1_scl: track 0.00 -> 42.3 mm, vias 0 -> 2
- net /i2c1_sda: track 0.00 -> 42.0 mm, vias 0 -> 4
- net Net-(J8-Pad3): track 0.00 -> 41.9 mm, vias 0 -> 1
- net /adc_v: track 0.00 -> 40.3 mm, vias 0 -> 2
- net Net-(J11-Pad3): track 0.00 -> 32.9 mm, vias 0 -> 1
- net Net-(J9-Pad3): track 0.00 -> 30.0 mm, vias 0 -> 1
- net +6V: track 66.3 -> 95.0 mm
- net /i2c0_scl: track 0.00 -> 24.9 mm, vias 0 -> 2
- net Net-(J15-Pin_3): track 0.00 -> 24.2 mm, vias 0 -> 2
- net /i2c0_sda: track 0.00 -> 21.1 mm, vias 0 -> 2
- net /mmc/3v3_filter: track 0.00 -> 17.9 mm, vias 0 -> 2
- net /bmp390/filter_3v3: track 0.00 -> 17.3 mm, vias 0 -> 2
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- added copper zone on B.Cu, net GND
Other:
- board outline added: 100 x 70 mm
- board text added: "+3V3"
- board text added: "-"
- board text added: "6V"
- board text added: "Backup_I2C"
- board text added: "DiffPressure"
- board text added: "GND"
- board text added: "GP10"
- board text added: "GP11"
- board text added: "GP12"
- board text added: "GP2"
- board text added: "GP3"
- board text added: "GP8"
- board text added: "GP9"
- board text added: "GPS"
- board text added: "NC"
- board text added: "PWM"
- board text added: "RC_Antenna"
- board text added: "SCL"
- board text added: "SDA"

Commit message: feat: rev1 added sdcard
Parts:
- removed the IC3 at (159.9, 107.5)
- removed the J12 at (127.2, 101.1)
- added C32: 22u, Capacitor_SMD:C_0603_1608Metric, B.Cu at (131.0, 106.8)
- added C33: 100n, Capacitor_SMD:C_0603_1608Metric, B.Cu at (129.5, 106.8)
- added J14: 502570-0893, eng_plane_lib:5025700893, B.Cu at (119.8, 106.5)
- added J15: Conn_01x04_Pin, Connector_PinHeader_2.54mm:PinHeader_1x04_P2.54mm_Vertical, F.Cu at (127.7, 121.6)
- added R25: 10k, PCM_SparkFun-Resistor:R_0603_1608Metric, B.Cu at (130.2, 109.5)
- added R26: 22, PCM_SparkFun-Resistor:R_0603_1608Metric, F.Cu at (127.8, 108.5)
- added R27: 10k, PCM_SparkFun-Resistor:R_0603_1608Metric, B.Cu at (130.2, 112.5)
- added R28: 10k, PCM_SparkFun-Resistor:R_0603_1608Metric, B.Cu at (130.2, 103.0)
- added R29: 22, PCM_SparkFun-Resistor:R_0603_1608Metric, F.Cu at (127.8, 111.3)
- added R30: 10k, PCM_SparkFun-Resistor:R_0603_1608Metric, B.Cu at (130.2, 111.0)
- added R31: 10k, PCM_SparkFun-Resistor:R_0603_1608Metric, B.Cu at (130.2, 101.5)
- added U3: BMP581, eng_plane_lib:BMP581, F.Cu at (159.9, 107.5)
- C31: renamed from C30; value 1u -> 10u
- moved C25 0.18 mm to (159.7, 104.6)
- moved C26 0.10 mm to (162.9, 107.7)
- moved C27 0.09 mm to (165.3, 107.6)
- moved L4 0.06 mm to (167.7, 107.0)
- renumbered C31 to C29, C29 to C30, C7 to C6, C6 to C7, IC4 to IC3, J14 to J1, J8 to J10, J9 to J11, J10 to J12, J11 to J13, J15 to J2, J1 to J3, J2 to J4, J3 to J5, J4 to J6, J5 to J7, J6 to J8, J7 to J9, R22 to R1, R23 to R10, R7 to R11, R8 to R12, R9 to R13, R10 to R14, R11 to R15, R12 to R16, R13 to R17, R14 to R18, R15 to R19, R21 to R2, R16 to R20, R17 to R21, R18 to R22, R19 to R23, R20 to R24, R1 to R3, R2 to R4, R3 to R5, R4 to R6, R24 to R7, R5 to R8, R6 to R9
Connections:
- net /5v_div renamed /POWER/5v_div
- net /6v_div renamed /POWER/6v_div
- net /bmp390/filter_3v3 renamed /bmp581/filter_3v3
- A1 pad 11: Net-(A1-GPIO8) -> /spi1_rx
- A1 pad 12: Net-(A1-GPIO9) -> /spi1_cs
- A1 pad 14: Net-(A1-GPIO10) -> /spi1_sclk
- A1 pad 15: Net-(A1-GPIO11) -> /spi1_tx
- A1 pad 16: Net-(A1-GPIO12) -> /sd_int
- A1 pad 19: unconnected-(A1-GPIO14-Pad19) -> Net-(A1-GPIO14)
- A1 pad 20: unconnected-(A1-GPIO15-Pad20) -> Net-(A1-GPIO15)
Routing:
- net +3V3: track 183.2 -> 218.6 mm, vias 0 -> 1
- net /sd_int: track 0.00 -> 24.0 mm, vias 0 -> 1
- net /spi1_cs: track 0.00 -> 23.1 mm, vias 0 -> 1
- net /spi1_rx: track 0.00 -> 11.2 mm, vias 0 -> 1
- net Net-(J14-CMD): track 0.00 -> 10.3 mm, vias 0 -> 1
- net Net-(J14-DAT2): track 0.00 -> 6.60 mm
- net Net-(J14-CLK): track 0.00 -> 5.75 mm, vias 0 -> 1
- net Net-(J14-DAT1): track 0.00 -> 5.55 mm
- net Net-(A1-GPIO12): track 5.17 -> 0.00 mm
- net Net-(A1-GPIO11): track 5.17 -> 0.00 mm
- net Net-(A1-GPIO10): track 5.17 -> 0.00 mm
- net Net-(A1-GPIO9): track 4.20 -> 0.00 mm
- net Net-(A1-GPIO8): track 4.20 -> 0.00 mm
- net Net-(A1-GPIO15): track 0.00 -> 3.85 mm
- net Net-(A1-GPIO14): track 0.00 -> 3.85 mm
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Other:
- board text removed: "GP10"
- board text removed: "GP11"
- board text removed: "GP12"
- board text removed: "GP8"
- board text removed: "GP9"

Commit message: feat: new inductor.exe
Parts:
- L2: footprint Inductor_SMD:L_7.3x7.3_H4.5 -> eng_plane_lib:7447714220
- moved L2 1.45 mm to (198.2, 116.8), turned to -90 degrees
- moved R16 0.92 mm to (184.7, 114.3), turned to 0 degrees
- moved J5 0.82 mm to (207.0, 112.7)
- moved C3 0.34 mm to (186.2, 91.7)
- moved C14 0.28 mm to (188.5, 111.1)
Routing:
- net Net-(U2-SW): track 6.71 -> 22.6 mm, vias 0 -> 4
- net Net-(U1-SW): track 7.78 -> 21.5 mm, vias 0 -> 5
- net +5V: track 142.2 -> 150.2 mm
- net GND: track 32.0 -> 24.8 mm, vias 420 -> 400
- net VBATT: track 43.1 -> 45.0 mm
- net /POWER/6v_div: track 5.47 -> 6.47 mm
- added copper zone on F.Cu, net +5V

Commit message: feat: final changes, sent to prod
Parts:
- added C24: 0.1u, Capacitor_SMD:C_0603_1608Metric, F.Cu at (194.1, 80.8)
- added C32: 0.1u, Capacitor_SMD:C_0603_1608Metric, F.Cu at (190.9, 121.2)
- C18: renamed from C32; footprint Capacitor_SMD:C_0603_1608Metric -> Capacitor_SMD:C_1206_3216Metric
- C27: renamed from C10; footprint Capacitor_SMD:C_0603_1608Metric -> Capacitor_SMD:C_0805_2012Metric
- D3: renamed from D1; footprint Diode_SMD:D_SMA -> Diode_SMD:D_SMA-SMB_Universal_Handsoldering
- L1: renamed from L3; footprint PCM_SparkFun-Capacitor:C_0805_2012Metric -> PCM_SparkFun-Resistor:R_0603_1608Metric
- L2: renamed from L4; footprint PCM_SparkFun-Capacitor:C_0805_2012Metric -> PCM_SparkFun-Resistor:R_0603_1608Metric
- L3: renamed from L5; footprint PCM_SparkFun-Capacitor:C_0805_2012Metric -> PCM_SparkFun-Resistor:R_0603_1608Metric
- R11: renamed from R13; value 100 -> 22
- R12: renamed from R14; value 100 -> 22
- R13: renamed from R17; value 100 -> 22
- R14: renamed from R18; value 100 -> 22
- R15: renamed from R19; value 100 -> 22
- R16: renamed from R20; value 100 -> 22
- R6: renamed from R10; value 100 -> 22
- R8: renamed from R11; value 100 -> 22
- R9: renamed from R12; value 100 -> 22
- moved L3 5.27 mm to (121.8, 118.0)
- moved C17 5.21 mm to (119.2, 118.8)
- moved C34 4.59 mm to (186.3, 121.0)
- moved C18 1.70 mm to (132.6, 106.0), turned to 0 degrees
- moved D3 0.95 mm to (154.9, 81.7)
- moved C33 0.64 mm to (188.9, 121.0)
- moved C15 0.35 mm to (113.8, 118.7)
- moved R30 0.27 mm to (185.5, 116.8)
- moved C16 0.25 mm to (118.8, 123.9)
- moved C27 0.22 mm to (185.4, 83.2)
- moved C35 0.10 mm to (183.7, 116.8)
- renumbered C4 to C1, C24 to C10, C25 to C11, C26 to C12, C27 to C13, C28 to C14, C29 to C15, C30 to C16, C31 to C17, C33 to C19, C6 to C2, C1 to C20, C2 to C21, C3 to C22, C5 to C23, C7 to C25, C8 to C26, C12 to C28, C13 to C29, C20 to C3, C14 to C30, C17 to C31, C18 to C33, C19 to C34, C21 to C35, C9 to C4, C11 to C5, C15 to C6, C16 to C7, C22 to C8, C23 to C9, D3 to D1, J8 to J1, J9 to J10, J10 to J11, J11 to J12, J12 to J13, J13 to J14, J14 to J15, J1 to J2, J15 to J3, J2 to J4, J7 to J5, J4 to J6, J5 to J7, J6 to J8, J3 to J9, L1 to L4, L2 to L5, R4 to R10, R21 to R17, R22 to R18, R23 to R19, R24 to R20, R29 to R21, R25 to R22, R26 to R23, R27 to R24, R28 to R25, R30 to R26, R31 to R27, R5 to R28, R6 to R29, R8 to R3, R15 to R30, R16 to R31, R9 to R4, R7 to R5, R3 to R7, U3 to U1, U1 to U2, U2 to U3
Connections:
- C11 pad 2: /bmp581/filter_3v3 -> +3V3
- C16 pad 1: /mmc/3v3_filter -> +3V3
- C8 pad 2: /bmi270/filter_3v3 -> +3V3
- IC2 pad 12: /bmi270/filter_3v3 -> +3V3
- IC2 pad 5: /bmi270/filter_3v3 -> +3V3
- IC3 pad 13: /mmc/3v3_filter -> +3V3
- IC3 pad 4: /mmc/3v3_filter -> +3V3
- U1 pad 1: /bmp581/filter_3v3 -> +3V3
- U1 pad 6: /bmp581/filter_3v3 -> +3V3
Routing:
- net +3V3: track 218.6 -> 268.7 mm, vias 1 -> 5
- net GND: track 24.8 -> 0.04 mm, vias 400 -> 416
- net /bmi270/filter_3v3: track 16.8 -> 5.75 mm
- net /bmp581/filter_3v3: track 17.3 -> 6.31 mm, vias 2 -> 0
- net /mmc/3v3_filter: track 17.9 -> 9.56 mm
- net +5V: track 150.2 -> 154.4 mm
- net Net-(A1-VSYS): track 4.98 -> 4.43 mm
Other:
- board text added: "Maksymilian Książka Date: 06-08-2026 Version: 1.0 Revision: 1"
