File: bmi270.kicad_sch (KiCad schematic)
At the start: 5 parts, among them IC2 BMI270

Commit message: sisyphus goes hard, awaiting review.
Connections:
- net +3V3: no longer C22.2, IC2.12 (CSB), IC2.5 (VDDIO)
- net filter_3v3: now reaches C23.2, C24.1, IC2.8 (VDD), L3.1
- net filter_3v3: now also C22.2, IC2.12 (CSB), IC2.5 (VDDIO)
Changed lines of the file:
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@@
 	)
 	(junction
+		(at 130.81 74.93)
+		(diameter 0)
+		(color 0 0 0 0)
+	)
+	(junction
 		(at 111.76 95.25)
 		(diameter 0)
@@
 	)
 	(junction
+		(at 133.35 74.93)
+		(diameter 0)
+		(color 0 0 0 0)
+	)
+	(junction
 		(at 127 74.93)
 		(diameter 0)
@@
 	(wire
 		(pts
+			(xy 113.03 48.26) (xy 130.81 48.26)
+		)
+		(stroke
+			(width 0)
+			(type default)
+		)
+	)
+	(wire
+		(pts
 			(xy 113.03 52.07) (xy 113.03 48.26)
 		)
@@
 	(wire
 		(pts
+			(xy 133.35 102.87) (xy 133.35 74.93)
+		)
+		(stroke
+			(width 0)
+			(type default)
+		)
+	)
+	(wire
+		(pts
+			(xy 130.81 74.93) (xy 133.35 74.93)
+		)
+		(stroke
+			(width 0)
+			(type default)
+		)
+	)
+	(wire
+		(pts
 			(xy 113.03 95.25) (xy 113.03 92.71)
 		)
@@
 	(wire
 		(pts
+			(xy 107.95 102.87) (xy 133.35 102.87)
+		)
+		(stroke
+			(width 0)
+			(type default)
+		)
+	)
+	(wire
+		(pts
 			(xy 110.49 92.71) (xy 110.49 95.25)
 		)
@@
 	(wire
 		(pts
-			(xy 127 74.93) (xy 142.24 74.93)
+			(xy 133.35 74.93) (xy 142.24 74.93)
+		)
+		(stroke
+			(width 0)
+			(type default)
+		)
+	)
+	(wire
+		(pts
+			(xy 130.81 48.26) (xy 130.81 74.93)
+		)
+		(stroke
+			(width 0)
+			(type default)
+		)
+	)
+	(wire
+		(pts
+			(xy 127 74.93) (xy 130.81 74.93)
 		)
 		(stroke
@@
 		)
 	)
+	(label "filter_3v3"
+		(at 130.81 48.26 0)
+		(effects
+			(font
+				(size 1.27 1.27)
+			)
+			(justify left bottom)
+		)
+	)
 	(hierarchical_label "BMI_SDA"
 		(shape bidirectional)
@@
 		(dnp no)
 		(fields_autoplaced yes)
-		(property "Reference" "#PWR040"
+		(property "Reference" "#PWR042"
 			(at 142.24 88.9 0)
 			(hide yes)
@@
 			(project "engineering_plane"
 				(path "/f9a2ded0-d803-4be9-b2f5-4dda0f6b4d9a/a759a096-c40b-4f10-8a53-3aaa1ae105c2"
-					(reference "#PWR040")
-					(unit 1)
-				)
-			)
-		)
-	)
-	(symbol
-		(lib_id "power:+3V3")
-		(at 113.03 48.26 0)
-		(unit 1)
-		(body_style 1)
-		(exclude_from_sim no)
-		(in_bom yes)
-		(on_board yes)
-		(in_pos_files yes)
-		(dnp no)
-		(fields_autoplaced yes)
-		(property "Reference" "#PWR038"
-			(at 113.03 52.07 0)
-			(hide yes)
-			(show_name no)
-			(do_not_autoplace no)
-			(effects
-				(font
-					(size 1.27 1.27)
-				)
-			)
-		)
-		(property "Value" "+3V3"
-			(at 113.03 43.18 0)
-			(show_name no)
-			(do_not_autoplace no)
-			(effects
-				(font
-					(size 1.27 1.27)
-				)
-			)
-		)
-		(property "Footprint" ""
-			(at 113.03 48.26 0)
-			(hide yes)
-			(show_name no)
-			(do_not_autoplace no)
-			(effects
-				(font
-					(size 1.27 1.27)
-				)
-			)
-		)
-		(property "Datasheet" ""
-			(at 113.03 48.26 0)
-			(hide yes)
-			(show_name no)
-			(do_not_autoplace no)
-			(effects
-				(font
-					(size 1.27 1.27)
-				)
-			)
-		)
-		(property "Description" "Power symbol creates a global label with name \"+3V3\""
-			(at 113.03 48.26 0)
-			(hide yes)
-			(show_name no)
-			(do_not_autoplace no)
-			(effects
-				(font
-					(size 1.27 1.27)
-				)
-			)
-		)
-		(pin "1"
-		)
-		(instances
-			(project "engineering_plane"
-				(path "/f9a2ded0-d803-4be9-b2f5-4dda0f6b4d9a/a759a096-c40b-4f10-8a53-3aaa1ae105c2"
-					(reference "#PWR038")
+					(reference "#PWR042")
 					(unit 1)
 				)
@@
 		(dnp no)
 		(fields_autoplaced yes)
-		(property "Reference" "#PWR037"
+		(property "Reference" "#PWR040"
 			(at 111.76 101.6 0)
 			(hide yes)
@@
 			(project "engineering_plane"
 				(path "/f9a2ded0-d803-4be9-b2f5-4dda0f6b4d9a/a759a096-c40b-4f10-8a53-3aaa1ae105c2"
-					(reference "#PWR037")
+					(reference "#PWR040")
 					(unit 1)
 				)
@@
 	)
 	(symbol
-		(lib_id "power:+3V3")
-		(at 107.95 102.87 90)
-		(unit 1)
-		(body_style 1)
-		(exclude_from_sim no)
-		(in_bom yes)
-		(on_board yes)
-		(in_pos_files yes)
-		(dnp no)
-		(fields_autoplaced yes)
-		(property "Reference" "#PWR036"
-			(at 111.76 102.87 0)
-			(hide yes)
-			(show_name no)
-			(do_not_autoplace no)
-			(effects
-				(font
-					(size 1.27 1.27)
-				)
-			)
-		)
-		(property "Value" "+3V3"
-			(at 104.14 102.8699 90)
-			(show_name no)
-			(do_not_autoplace no)
-			(effects
-				(font
-					(size 1.27 1.27)
-				)
-				(justify left)
-			)
-		)
-		(property "Footprint" ""
-			(at 107.95 102.87 0)
-			(hide yes)
-			(show_name no)
-			(do_not_autoplace no)
-			(effects
-				(font
-					(size 1.27 1.27)
-				)
-			)
-		)
-		(property "Datasheet" ""
-			(at 107.95 102.87 0)
-			(hide yes)
-			(show_name no)
-			(do_not_autoplace no)
-			(effects
-				(font
-					(size 1.27 1.27)
-				)
-			)
-		)
-		(property "Description" "Power symbol creates a global label with name \"+3V3\""
-			(at 107.95 102.87 0)
-			(hide yes)
-			(show_name no)
-			(do_not_autoplace no)
-			(effects
-				(font
-					(size 1.27 1.27)
-				)
-			)
-		)
-		(pin "1"
-		)
-		(instances
-			(project "engineering_plane"
-				(path "/f9a2ded0-d803-4be9-b2f5-4dda0f6b4d9a/a759a096-c40b-4f10-8a53-3aaa1ae105c2"
-					(reference "#PWR036")
-					(unit 1)
-				)
-			)
-		)
-	)
-	(symbol
 		(lib_id "Device:C")
 		(at 142.24 78.74 0)
@@
 		(in_pos_files yes)
 		(dnp no)
-		(property "Reference" "#PWR041"
+		(property "Reference" "#PWR043"
 			(at 156.21 77.47 0)
 			(hide yes)
@@
 			(project "engineering_plane"
 				(path "/f9a2ded0-d803-4be9-b2f5-4dda0f6b4d9a/a759a096-c40b-4f10-8a53-3aaa1ae105c2"
-					(reference "#PWR041")
+					(reference "#PWR043")
 					(unit 1)
 				)
@@
 		(dnp no)
 		(fields_autoplaced yes)
-		(property "Reference" "#PWR035"
+		(property "Reference" "#PWR039"
 			(at 93.98 95.25 0)
 			(hide yes)
@@
 			(project "engineering_plane"
 				(path "/f9a2ded0-d803-4be9-b2f5-4dda0f6b4d9a/a759a096-c40b-4f10-8a53-3aaa1ae105c2"
-					(reference "#PWR035")
+					(reference "#PWR039")
 					(unit 1)
 				)
@@
 		(dnp no)
 		(fields_autoplaced yes)
-		(property "Reference" "#PWR039"
+		(property "Reference" "#PWR041"
 			(at 127 88.9 0)
 			(hide yes)
@@
 			(project "engineering_plane"
 				(path "/f9a2ded0-d803-4be9-b2f5-4dda0f6b4d9a/a759a096-c40b-4f10-8a53-3aaa1ae105c2"
-					(reference "#PWR039")
+					(reference "#PWR041")
 					(unit 1)
 				)
@@
 		(dnp no)
 		(fields_autoplaced yes)
-		(property "Reference" "#PWR034"
+		(property "Reference" "#PWR038"
 			(at 88.9 67.31 0)
 			(hide yes)
@@
 			(project "engineering_plane"
 				(path "/f9a2ded0-d803-4be9-b2f5-4dda0f6b4d9a/a759a096-c40b-4f10-8a53-3aaa1ae105c2"
-					(reference "#PWR034")
+					(reference "#PWR038")
 					(unit 1)
 				)

Commit message: feat: rev1 added sdcard
Parts:
- C24: now not fitted
Changed lines of the file:
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@@
 		(dnp no)
 		(fields_autoplaced yes)
-		(property "Reference" "#PWR042"
+		(property "Reference" "#PWR052"
 			(at 142.24 88.9 0)
 			(hide yes)
@@
 		(instances
 			(project "engineering_plane"
-				(path "/f9a2ded0-d803-4be9-b2f5-4dda0f6b4d9a/a759a096-c40b-4f10-8a53-3aaa1ae105c2"
-					(reference "#PWR042")
+				(path "/f9a2ded0-d803-4be9-b2f5-4dda0f6b4d9a/d92f5ceb-a3bf-4490-a03e-54e85bc3d6ad"
+					(reference "#PWR052")
 					(unit 1)
 				)
@@
 		(dnp no)
 		(fields_autoplaced yes)
-		(property "Reference" "#PWR040"
+		(property "Reference" "#PWR050"
 			(at 111.76 101.6 0)
 			(hide yes)
@@
 		(instances
 			(project "engineering_plane"
-				(path "/f9a2ded0-d803-4be9-b2f5-4dda0f6b4d9a/a759a096-c40b-4f10-8a53-3aaa1ae105c2"
-					(reference "#PWR040")
+				(path "/f9a2ded0-d803-4be9-b2f5-4dda0f6b4d9a/d92f5ceb-a3bf-4490-a03e-54e85bc3d6ad"
+					(reference "#PWR050")
 					(unit 1)
 				)
@@
 		(instances
 			(project "engineering_plane"
-				(path "/f9a2ded0-d803-4be9-b2f5-4dda0f6b4d9a/a759a096-c40b-4f10-8a53-3aaa1ae105c2"
+				(path "/f9a2ded0-d803-4be9-b2f5-4dda0f6b4d9a/d92f5ceb-a3bf-4490-a03e-54e85bc3d6ad"
 					(reference "IC2")
 					(unit 1)
@@
 		(on_board yes)
 		(in_pos_files yes)
-		(dnp no)
+		(dnp yes)
 		(property "Reference" "C24"
 			(at 135.382 77.978 0)
@@
 		(instances
 			(project "engineering_plane"
-				(path "/f9a2ded0-d803-4be9-b2f5-4dda0f6b4d9a/a759a096-c40b-4f10-8a53-3aaa1ae105c2"
+				(path "/f9a2ded0-d803-4be9-b2f5-4dda0f6b4d9a/d92f5ceb-a3bf-4490-a03e-54e85bc3d6ad"
 					(reference "C24")
 					(unit 1)
@@
 		(in_pos_files yes)
 		(dnp no)
-		(property "Reference" "#PWR043"
+		(property "Reference" "#PWR053"
 			(at 156.21 77.47 0)
 			(hide yes)
@@
 		(instances
 			(project "engineering_plane"
-				(path "/f9a2ded0-d803-4be9-b2f5-4dda0f6b4d9a/a759a096-c40b-4f10-8a53-3aaa1ae105c2"
-					(reference "#PWR043")
+				(path "/f9a2ded0-d803-4be9-b2f5-4dda0f6b4d9a/d92f5ceb-a3bf-4490-a03e-54e85bc3d6ad"
+					(reference "#PWR053")
 					(unit 1)
 				)
@@
 		(instances
 			(project "engineering_plane"
-				(path "/f9a2ded0-d803-4be9-b2f5-4dda0f6b4d9a/a759a096-c40b-4f10-8a53-3aaa1ae105c2"
+				(path "/f9a2ded0-d803-4be9-b2f5-4dda0f6b4d9a/d92f5ceb-a3bf-4490-a03e-54e85bc3d6ad"
 					(reference "C22")
 					(unit 1)
@@
 		(dnp no)
 		(fields_autoplaced yes)
-		(property "Reference" "#PWR039"
+		(property "Reference" "#PWR049"
 			(at 93.98 95.25 0)
 			(hide yes)
@@
 		(instances
 			(project "engineering_plane"
-				(path "/f9a2ded0-d803-4be9-b2f5-4dda0f6b4d9a/a759a096-c40b-4f10-8a53-3aaa1ae105c2"
-					(reference "#PWR039")
+				(path "/f9a2ded0-d803-4be9-b2f5-4dda0f6b4d9a/d92f5ceb-a3bf-4490-a03e-54e85bc3d6ad"
+					(reference "#PWR049")
 					(unit 1)
 				)
@@
 		(instances
 			(project "engineering_plane"
-				(path "/f9a2ded0-d803-4be9-b2f5-4dda0f6b4d9a/a759a096-c40b-4f10-8a53-3aaa1ae105c2"
+				(path "/f9a2ded0-d803-4be9-b2f5-4dda0f6b4d9a/d92f5ceb-a3bf-4490-a03e-54e85bc3d6ad"
 					(reference "L3")
 					(unit 1)
@@
 		(dnp no)
 		(fields_autoplaced yes)
-		(property "Reference" "#PWR041"
+		(property "Reference" "#PWR051"
 			(at 127 88.9 0)
 			(hide yes)
@@
 		(instances
 			(project "engineering_plane"
-				(path "/f9a2ded0-d803-4be9-b2f5-4dda0f6b4d9a/a759a096-c40b-4f10-8a53-3aaa1ae105c2"
-					(reference "#PWR041")
+				(path "/f9a2ded0-d803-4be9-b2f5-4dda0f6b4d9a/d92f5ceb-a3bf-4490-a03e-54e85bc3d6ad"
+					(reference "#PWR051")
 					(unit 1)
 				)
@@
 		(instances
 			(project "engineering_plane"
-				(path "/f9a2ded0-d803-4be9-b2f5-4dda0f6b4d9a/a759a096-c40b-4f10-8a53-3aaa1ae105c2"
+				(path "/f9a2ded0-d803-4be9-b2f5-4dda0f6b4d9a/d92f5ceb-a3bf-4490-a03e-54e85bc3d6ad"
 					(reference "C23")
 					(unit 1)
@@
 		(dnp no)
 		(fields_autoplaced yes)
-		(property "Reference" "#PWR038"
+		(property "Reference" "#PWR048"
 			(at 88.9 67.31 0)
 			(hide yes)
@@
 		(instances
 			(project "engineering_plane"
-				(path "/f9a2ded0-d803-4be9-b2f5-4dda0f6b4d9a/a759a096-c40b-4f10-8a53-3aaa1ae105c2"
-					(reference "#PWR038")
-					(unit 1)
-				)
+				(path "/f9a2ded0-d803-4be9-b2f5-4dda0f6b4d9a/d92f5ceb-a3bf-4490-a03e-54e85bc3d6ad"
+					(reference "#PWR048")
+					(unit 1)
+				)

Commit message: feat: final changes, sent to prod
Parts:
- L1: renamed from L3; footprint PCM_SparkFun-Capacitor:C_0805_2012Metric -> PCM_SparkFun-Resistor:R_0603_1608Metric
- renumbered C24 to C10, C22 to C8, C23 to C9
Connections:
- net +3V3: now also C8.2, IC2.12 (CSB), IC2.5 (VDDIO)
- net filter_3v3: no longer C8.2, IC2.12 (CSB), IC2.5 (VDDIO)
Changed lines of the file:
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@@
 	)
 	(junction
-		(at 107.95 95.25)
+		(at 152.4 74.93)
 		(diameter 0)
 		(color 0 0 0 0)
 	)
 	(junction
-		(at 130.81 74.93)
+		(at 156.21 74.93)
 		(diameter 0)
 		(color 0 0 0 0)
 	)
 	(junction
-		(at 111.76 95.25)
+		(at 107.95 95.25)
 		(diameter 0)
 		(color 0 0 0 0)
 	)
 	(junction
-		(at 133.35 74.93)
+		(at 111.76 95.25)
 		(diameter 0)
 		(color 0 0 0 0)
@@
 	(wire
 		(pts
-			(xy 113.03 48.26) (xy 130.81 48.26)
+			(xy 152.4 74.93) (xy 149.86 74.93)
 		)
 		(stroke
@@
 	(wire
 		(pts
-			(xy 113.03 52.07) (xy 113.03 48.26)
+			(xy 113.03 48.26) (xy 152.4 48.26)
 		)
 		(stroke
@@
 	(wire
 		(pts
-			(xy 125.73 74.93) (xy 127 74.93)
+			(xy 113.03 52.07) (xy 113.03 48.26)
 		)
 		(stroke
@@
 	(wire
 		(pts
-			(xy 111.76 95.25) (xy 113.03 95.25)
+			(xy 125.73 74.93) (xy 127 74.93)
 		)
 		(stroke
@@
 	(wire
 		(pts
-			(xy 142.24 74.93) (xy 144.78 74.93)
+			(xy 111.76 95.25) (xy 113.03 95.25)
 		)
 		(stroke
@@
 	(wire
 		(pts
-			(xy 107.95 95.25) (xy 107.95 102.87)
+			(xy 142.24 74.93) (xy 144.78 74.93)
 		)
 		(stroke
@@
 	(wire
 		(pts
-			(xy 133.35 102.87) (xy 133.35 74.93)
+			(xy 107.95 95.25) (xy 107.95 102.87)
 		)
 		(stroke
@@
 	(wire
 		(pts
-			(xy 130.81 74.93) (xy 133.35 74.93)
+			(xy 113.03 95.25) (xy 113.03 92.71)
 		)
 		(stroke
@@
 	(wire
 		(pts
-			(xy 113.03 95.25) (xy 113.03 92.71)
+			(xy 107.95 102.87) (xy 156.21 102.87)
 		)
 		(stroke
@@
 	(wire
 		(pts
-			(xy 107.95 102.87) (xy 133.35 102.87)
+			(xy 156.21 102.87) (xy 156.21 74.93)
 		)
 		(stroke
@@
 	(wire
 		(pts
-			(xy 156.21 74.93) (xy 149.86 74.93)
+			(xy 156.21 74.93) (xy 152.4 74.93)
 		)
 		(stroke
@@
 	(wire
 		(pts
-			(xy 133.35 74.93) (xy 142.24 74.93)
-		)
-		(stroke
-			(width 0)
-			(type default)
-		)
-	)
-	(wire
-		(pts
-			(xy 130.81 48.26) (xy 130.81 74.93)
+			(xy 152.4 48.26) (xy 152.4 74.93)
 		)
 		(stroke
@@
 	(wire
 		(pts
-			(xy 127 74.93) (xy 130.81 74.93)
+			(xy 127 74.93) (xy 142.24 74.93)
 		)
 		(stroke
@@
 	)
 	(label "filter_3v3"
-		(at 130.81 48.26 0)
+		(at 133.35 74.93 0)
 		(effects
 			(font
@@
 		(dnp no)
 		(fields_autoplaced yes)
-		(property "Reference" "#PWR052"
+		(property "Reference" "#PWR042"
 			(at 142.24 88.9 0)
 			(hide yes)
@@
 			(project "engineering_plane"
 				(path "/f9a2ded0-d803-4be9-b2f5-4dda0f6b4d9a/d92f5ceb-a3bf-4490-a03e-54e85bc3d6ad"
-					(reference "#PWR052")
+					(reference "#PWR042")
 					(unit 1)
 				)
@@
 		(dnp no)
 		(fields_autoplaced yes)
-		(property "Reference" "#PWR050"
+		(property "Reference" "#PWR040"
 			(at 111.76 101.6 0)
 			(hide yes)
@@
 			(project "engineering_plane"
 				(path "/f9a2ded0-d803-4be9-b2f5-4dda0f6b4d9a/d92f5ceb-a3bf-4490-a03e-54e85bc3d6ad"
-					(reference "#PWR050")
+					(reference "#PWR040")
 					(unit 1)
 				)
@@
 		(in_pos_files yes)
 		(dnp yes)
-		(property "Reference" "C24"
+		(property "Reference" "C10"
 			(at 135.382 77.978 0)
 			(show_name no)
@@
 			(project "engineering_plane"
 				(path "/f9a2ded0-d803-4be9-b2f5-4dda0f6b4d9a/d92f5ceb-a3bf-4490-a03e-54e85bc3d6ad"
-					(reference "C24")
+					(reference "C10")
 					(unit 1)
 				)
@@
 		(in_pos_files yes)
 		(dnp no)
-		(property "Reference" "#PWR053"
+		(property "Reference" "#PWR043"
 			(at 156.21 77.47 0)
 			(hide yes)
@@
 			(project "engineering_plane"
 				(path "/f9a2ded0-d803-4be9-b2f5-4dda0f6b4d9a/d92f5ceb-a3bf-4490-a03e-54e85bc3d6ad"
-					(reference "#PWR053")
+					(reference "#PWR043")
 					(unit 1)
 				)
@@
 		(in_pos_files yes)
 		(dnp no)
-		(property "Reference" "C22"
+		(property "Reference" "C8"
 			(at 103.632 88.9 90)
 			(show_name no)
@@
 			(project "engineering_plane"
 				(path "/f9a2ded0-d803-4be9-b2f5-4dda0f6b4d9a/d92f5ceb-a3bf-4490-a03e-54e85bc3d6ad"
-					(reference "C22")
+					(reference "C8")
 					(unit 1)
 				)
@@
 		(dnp no)
 		(fields_autoplaced yes)
-		(property "Reference" "#PWR049"
+		(property "Reference" "#PWR039"
 			(at 93.98 95.25 0)
 			(hide yes)
@@
 			(project "engineering_plane"
 				(path "/f9a2ded0-d803-4be9-b2f5-4dda0f6b4d9a/d92f5ceb-a3bf-4490-a03e-54e85bc3d6ad"
-					(reference "#PWR049")
+					(reference "#PWR039")
 					(unit 1)
 				)
@@
 		(in_pos_files yes)
 		(dnp no)
-		(property "Reference" "L3"
+		(property "Reference" "L1"
 			(at 147.32 67.056 0)
 			(show_name no)
@@
 			)
 		)
-		(property "Footprint" "PCM_SparkFun-Capacitor:C_0805_2012Metric"
+		(property "Footprint" "PCM_SparkFun-Resistor:R_0603_1608Metric"
 			(at 147.32 86.36 0)
 			(hide yes)
@@
 			(project "engineering_plane"
 				(path "/f9a2ded0-d803-4be9-b2f5-4dda0f6b4d9a/d92f5ceb-a3bf-4490-a03e-54e85bc3d6ad"
-					(reference "L3")
+					(reference "L1")
 					(unit 1)
 				)
@@
 		(dnp no)
 		(fields_autoplaced yes)
-		(property "Reference" "#PWR051"
+		(property "Reference" "#PWR041"
 			(at 127 88.9 0)
 			(hide yes)
@@
 			(project "engineering_plane"
 				(path "/f9a2ded0-d803-4be9-b2f5-4dda0f6b4d9a/d92f5ceb-a3bf-4490-a03e-54e85bc3d6ad"
-					(reference "#PWR051")
+					(reference "#PWR041")
 					(unit 1)
 				)
@@
 		(in_pos_files yes)
 		(dnp no)
-		(property "Reference" "C23"
+		(property "Reference" "C9"
 			(at 131.826 78.486 0)
 			(show_name no)
@@
 			(project "engineering_plane"
 				(path "/f9a2ded0-d803-4be9-b2f5-4dda0f6b4d9a/d92f5ceb-a3bf-4490-a03e-54e85bc3d6ad"
-					(reference "C23")
+					(reference "C9")
 					(unit 1)
 				)
@@
 		(dnp no)
 		(fields_autoplaced yes)
-		(property "Reference" "#PWR048"
+		(property "Reference" "#PWR038"
 			(at 88.9 67.31 0)
 			(hide yes)
@@
 			(project "engineering_plane"
 				(path "/f9a2ded0-d803-4be9-b2f5-4dda0f6b4d9a/d92f5ceb-a3bf-4490-a03e-54e85bc3d6ad"
-					(reference "#PWR048")
+					(reference "#PWR038")
 					(unit 1)
 				)

Commit message: Revised componenents, need to route
Parts:
- removed C10: 1u, Capacitor_SMD:C_0603_1608Metric, symbol Device:C
- removed C8, C9: 100n, Capacitor_SMD:C_0603_1608Metric, symbol Device:C
- removed L1: 600 Ohm, PCM_SparkFun-Resistor:R_0603_1608Metric, symbol PCM_SparkFun-Coil:Ferrite_600Ohm_0805_500mA
- added C201, C202: 100nF, PCM_JLCPCB:C_0402, symbol PCM_JLCPCB-Capacitors:0402,100nF,(2)
- added C203: 1uF, PCM_JLCPCB:C_0402, symbol PCM_JLCPCB-Capacitors:0402,1uF
- added FB201: (no value), PCM_JLCPCB:FB_0603, symbol PCM_JLCPCB-Inductors:Ferrite,0603
- added TP201, TP202: 1.0mm, PCM_SparkFun-Connector:TestPoint-1.0mm, symbol PCM_SparkFun-Connector:TestPoint_1.0mm
- renumbered IC2 to IC201
Connections:
- net +3V3: now also C201.1, FB201.2, TP201.1
- net GND: now also C201.2, C202.2, C203.2
- net filter_3v3: now also C202.1, C203.1, FB201.1, TP202.1
- net BMI_SCL renamed I2C.SCL
- net BMI_SDA renamed I2C.SDA
Other:
- moved on the sheet: IC201
