File: bmp581.kicad_sch (KiCad schematic)
At the start: 5 parts, among them U3 BMP581

Commit message: feat: final changes, sent to prod
Parts:
- L2: renamed from L4; footprint PCM_SparkFun-Capacitor:C_0805_2012Metric -> PCM_SparkFun-Resistor:R_0603_1608Metric
- renumbered C25 to C11, C26 to C12, C27 to C13, U3 to U1
Connections:
- net +3V3: now also C11.2, U1.1 (VDDIO), U1.6 (CSB)
- net filter_3v3: no longer C11.2, U1.1 (VDDIO), U1.6 (CSB)
Changed lines of the file:
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@@
-	)
-	(junction
-		(at 116.84 78.74)
-		(diameter 0)
-		(color 0 0 0 0)
 	)
 	(junction
@@
 	)
 	(junction
+		(at 138.43 78.74)
+		(diameter 0)
+		(color 0 0 0 0)
+	)
+	(junction
 		(at 127 78.74)
 		(diameter 0)
 		(color 0 0 0 0)
 	)
-	(junction
-		(at 115.57 78.74)
-		(diameter 0)
-		(color 0 0 0 0)
-	)
 	(wire
 		(pts
-			(xy 111.76 78.74) (xy 115.57 78.74)
+			(xy 138.43 57.15) (xy 138.43 105.41)
 		)
 		(stroke
@@
 	(wire
 		(pts
-			(xy 116.84 105.41) (xy 116.84 78.74)
+			(xy 81.28 96.52) (xy 81.28 105.41)
 		)
 		(stroke
@@
 	(wire
 		(pts
-			(xy 81.28 96.52) (xy 81.28 105.41)
+			(xy 62.23 83.82) (xy 63.5 83.82)
 		)
 		(stroke
@@
 	(wire
 		(pts
-			(xy 115.57 57.15) (xy 115.57 78.74)
+			(xy 102.87 83.82) (xy 101.6 83.82)
 		)
 		(stroke
@@
 	(wire
 		(pts
-			(xy 62.23 83.82) (xy 63.5 83.82)
+			(xy 138.43 78.74) (xy 134.62 78.74)
 		)
 		(stroke
@@
 	(wire
 		(pts
-			(xy 115.57 78.74) (xy 116.84 78.74)
+			(xy 83.82 57.15) (xy 138.43 57.15)
 		)
 		(stroke
@@
 	(wire
 		(pts
-			(xy 102.87 83.82) (xy 101.6 83.82)
+			(xy 102.87 81.28) (xy 102.87 83.82)
 		)
 		(stroke
@@
 	(wire
 		(pts
-			(xy 83.82 57.15) (xy 115.57 57.15)
+			(xy 101.6 78.74) (xy 111.76 78.74)
 		)
 		(stroke
@@
 	(wire
 		(pts
-			(xy 102.87 81.28) (xy 102.87 83.82)
+			(xy 127 78.74) (xy 129.54 78.74)
 		)
 		(stroke
@@
 	(wire
 		(pts
-			(xy 101.6 78.74) (xy 111.76 78.74)
+			(xy 62.23 78.74) (xy 63.5 78.74)
 		)
 		(stroke
@@
 	(wire
 		(pts
-			(xy 127 78.74) (xy 129.54 78.74)
+			(xy 140.97 78.74) (xy 138.43 78.74)
 		)
 		(stroke
@@
 	(wire
 		(pts
-			(xy 62.23 78.74) (xy 63.5 78.74)
+			(xy 83.82 57.15) (xy 83.82 66.04)
 		)
 		(stroke
@@
 	(wire
 		(pts
-			(xy 140.97 78.74) (xy 134.62 78.74)
+			(xy 62.23 81.28) (xy 63.5 81.28)
 		)
 		(stroke
@@
 	(wire
 		(pts
-			(xy 83.82 57.15) (xy 83.82 66.04)
+			(xy 81.28 105.41) (xy 138.43 105.41)
 		)
 		(stroke
@@
 	(wire
 		(pts
-			(xy 62.23 81.28) (xy 63.5 81.28)
-		)
-		(stroke
-			(width 0)
-			(type default)
-		)
-	)
-	(wire
-		(pts
-			(xy 81.28 105.41) (xy 116.84 105.41)
-		)
-		(stroke
-			(width 0)
-			(type default)
-		)
-	)
-	(wire
-		(pts
-			(xy 116.84 78.74) (xy 127 78.74)
+			(xy 111.76 78.74) (xy 127 78.74)
 		)
 		(stroke
@@
 	)
 	(label "filter_3v3"
-		(at 115.57 57.15 0)
+		(at 107.95 78.74 0)
 		(effects
 			(font
@@
 		(dnp no)
 		(fields_autoplaced yes)
-		(property "Reference" "#PWR059"
+		(property "Reference" "#PWR049"
 			(at 127 92.71 0)
 			(hide yes)
@@
 			(project "engineering_plane"
 				(path "/f9a2ded0-d803-4be9-b2f5-4dda0f6b4d9a/225c3c49-48ba-4300-a655-407153bb93d3"
-					(reference "#PWR059")
+					(reference "#PWR049")
 					(unit 1)
 				)
@@
 		(in_pos_files yes)
 		(dnp no)
-		(property "Reference" "L4"
+		(property "Reference" "L2"
 			(at 132.08 70.866 0)
 			(show_name no)
@@
 			)
 		)
-		(property "Footprint" "PCM_SparkFun-Capacitor:C_0805_2012Metric"
+		(property "Footprint" "PCM_SparkFun-Resistor:R_0603_1608Metric"
 			(at 132.08 90.17 0)
 			(hide yes)
@@
 			(project "engineering_plane"
 				(path "/f9a2ded0-d803-4be9-b2f5-4dda0f6b4d9a/225c3c49-48ba-4300-a655-407153bb93d3"
-					(reference "L4")
+					(reference "L2")
 					(unit 1)
 				)
@@
 		(in_pos_files yes)
 		(dnp no)
-		(property "Reference" "C26"
+		(property "Reference" "C12"
 			(at 116.586 82.296 0)
 			(show_name no)
@@
 			(project "engineering_plane"
 				(path "/f9a2ded0-d803-4be9-b2f5-4dda0f6b4d9a/225c3c49-48ba-4300-a655-407153bb93d3"
-					(reference "C26")
+					(reference "C12")
 					(unit 1)
 				)
@@
 		(dnp no)
 		(fields_autoplaced yes)
-		(property "Reference" "U3"
+		(property "Reference" "U1"
 			(at 86.9381 66.04 90)
 			(show_name no)
@@
 			(project "engineering_plane"
 				(path "/f9a2ded0-d803-4be9-b2f5-4dda0f6b4d9a/225c3c49-48ba-4300-a655-407153bb93d3"
-					(reference "U3")
+					(reference "U1")
 					(unit 1)
 				)
@@
 		(dnp no)
 		(fields_autoplaced yes)
-		(property "Reference" "#PWR054"
+		(property "Reference" "#PWR044"
 			(at 55.88 78.74 0)
 			(hide yes)
@@
 			(project "engineering_plane"
 				(path "/f9a2ded0-d803-4be9-b2f5-4dda0f6b4d9a/225c3c49-48ba-4300-a655-407153bb93d3"
-					(reference "#PWR054")
+					(reference "#PWR044")
 					(unit 1)
 				)
@@
 		(dnp no)
 		(fields_autoplaced yes)
-		(property "Reference" "#PWR056"
+		(property "Reference" "#PWR046"
 			(at 97.79 66.04 0)
 			(hide yes)
@@
 			(project "engineering_plane"
 				(path "/f9a2ded0-d803-4be9-b2f5-4dda0f6b4d9a/225c3c49-48ba-4300-a655-407153bb93d3"
-					(reference "#PWR056")
+					(reference "#PWR046")
 					(unit 1)
 				)
@@
 		(dnp no)
 		(fields_autoplaced yes)
-		(property "Reference" "#PWR058"
+		(property "Reference" "#PWR048"
 			(at 111.76 92.71 0)
 			(hide yes)
@@
 			(project "engineering_plane"
 				(path "/f9a2ded0-d803-4be9-b2f5-4dda0f6b4d9a/225c3c49-48ba-4300-a655-407153bb93d3"
-					(reference "#PWR058")
+					(reference "#PWR048")
 					(unit 1)
 				)
@@
 		(in_pos_files yes)
 		(dnp no)
-		(property "Reference" "C25"
+		(property "Reference" "C11"
 			(at 87.376 61.214 0)
 			(show_name no)
@@
 			(project "engineering_plane"
 				(path "/f9a2ded0-d803-4be9-b2f5-4dda0f6b4d9a/225c3c49-48ba-4300-a655-407153bb93d3"
-					(reference "C25")
+					(reference "C11")
 					(unit 1)
 				)
@@
 		(dnp no)
 		(fields_autoplaced yes)
-		(property "Reference" "#PWR057"
+		(property "Reference" "#PWR047"
 			(at 102.87 92.71 0)
 			(hide yes)
@@
 			(project "engineering_plane"
 				(path "/f9a2ded0-d803-4be9-b2f5-4dda0f6b4d9a/225c3c49-48ba-4300-a655-407153bb93d3"
-					(reference "#PWR057")
+					(reference "#PWR047")
 					(unit 1)
 				)
@@
 		(in_pos_files yes)
 		(dnp no)
-		(property "Reference" "#PWR060"
+		(property "Reference" "#PWR050"
 			(at 140.97 81.28 0)
 			(hide yes)
@@
 			(project "engineering_plane"
 				(path "/f9a2ded0-d803-4be9-b2f5-4dda0f6b4d9a/225c3c49-48ba-4300-a655-407153bb93d3"
-					(reference "#PWR060")
+					(reference "#PWR050")
 					(unit 1)
 				)
@@
 		(dnp no)
 		(fields_autoplaced yes)
-		(property "Reference" "#PWR055"
+		(property "Reference" "#PWR045"
 			(at 55.88 83.82 0)
 			(hide yes)
@@
 			(project "engineering_plane"
 				(path "/f9a2ded0-d803-4be9-b2f5-4dda0f6b4d9a/225c3c49-48ba-4300-a655-407153bb93d3"
-					(reference "#PWR055")
+					(reference "#PWR045")
 					(unit 1)
 				)
@@
 		(in_pos_files yes)
 		(dnp yes)
-		(property "Reference" "C27"
+		(property "Reference" "C13"
 			(at 120.142 81.788 0)
 			(show_name no)
@@
 			(project "engineering_plane"
 				(path "/f9a2ded0-d803-4be9-b2f5-4dda0f6b4d9a/225c3c49-48ba-4300-a655-407153bb93d3"
-					(reference "C27")
+					(reference "C13")
 					(unit 1)
 				)

Commit message: Revised componenents, need to route
Parts:
- removed C11, C12: 100n, Capacitor_SMD:C_0603_1608Metric, symbol Device:C
- removed C13: 1u, Capacitor_SMD:C_0603_1608Metric, symbol Device:C
- removed L2: 600 Ohm, PCM_SparkFun-Resistor:R_0603_1608Metric, symbol PCM_SparkFun-Coil:Ferrite_600Ohm_0805_500mA
- added C301, C302: 100nF, PCM_JLCPCB:C_0402, symbol PCM_JLCPCB-Capacitors:0402,100nF,(2)
- added C303: 1uF, PCM_JLCPCB:C_0402, symbol PCM_JLCPCB-Capacitors:0402,1uF
- added FB301: (no value), PCM_JLCPCB:FB_0603, symbol PCM_JLCPCB-Inductors:Ferrite,0603
- renumbered U1 to U301
Connections:
- net +3V3: now also C301.1, FB301.2
- net GND: now also C301.2, C302.2, C303.2
- net filter_3v3: now also C302.1, C303.1, FB301.1
- net bmp_SCL renamed I2C.SCL
- net bmp_SDA renamed I2C.SDA
Other:
- moved on the sheet: U301
