File: sd.kicad_sch (KiCad schematic)
At the start: 10 parts, among them J14 502570-0893

Commit message: feat: final changes, sent to prod
Parts:
- C18: renamed from C32; footprint Capacitor_SMD:C_0603_1608Metric -> Capacitor_SMD:C_1206_3216Metric
- renumbered C33 to C19, J14 to J15, R29 to R21, R25 to R22, R26 to R23, R27 to R24, R28 to R25, R30 to R26, R31 to R27
Changed lines of the file:
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@@
 		(in_pos_files yes)
 		(dnp no)
-		(property "Reference" "C32"
+		(property "Reference" "C18"
 			(at 56.134 84.836 0)
 			(show_name no)
@@
 			)
 		)
-		(property "Footprint" "Capacitor_SMD:C_0603_1608Metric"
+		(property "Footprint" "Capacitor_SMD:C_1206_3216Metric"
 			(at 61.9252 85.09 0)
 			(hide yes)
@@
 			(project "engineering_plane"
 				(path "/f9a2ded0-d803-4be9-b2f5-4dda0f6b4d9a/9c29d4f9-b687-4678-a7ec-dae4a703e307"
-					(reference "C32")
+					(reference "C18")
 					(unit 1)
 				)
@@
 		(dnp no)
 		(fields_autoplaced yes)
-		(property "Reference" "J14"
+		(property "Reference" "J15"
 			(at 123.19 62.23 0)
 			(show_name no)
@@
 			(project "engineering_plane"
 				(path "/f9a2ded0-d803-4be9-b2f5-4dda0f6b4d9a/9c29d4f9-b687-4678-a7ec-dae4a703e307"
-					(reference "J14")
+					(reference "J15")
 					(unit 1)
 				)
@@
 		(in_pos_files yes)
 		(dnp no)
-		(property "Reference" "R26"
+		(property "Reference" "R23"
 			(at 85.09 83.312 0)
 			(show_name no)
@@
 			(project "engineering_plane"
 				(path "/f9a2ded0-d803-4be9-b2f5-4dda0f6b4d9a/9c29d4f9-b687-4678-a7ec-dae4a703e307"
-					(reference "R26")
+					(reference "R23")
 					(unit 1)
 				)
@@
 		(dnp no)
 		(fields_autoplaced yes)
-		(property "Reference" "R29"
+		(property "Reference" "R21"
 			(at 77.47 68.58 0)
 			(show_name no)
@@
 			(project "engineering_plane"
 				(path "/f9a2ded0-d803-4be9-b2f5-4dda0f6b4d9a/9c29d4f9-b687-4678-a7ec-dae4a703e307"
-					(reference "R29")
+					(reference "R21")
 					(unit 1)
 				)
@@
 		(dnp no)
 		(fields_autoplaced yes)
-		(property "Reference" "R28"
+		(property "Reference" "R25"
 			(at 96.52 88.8999 90)
 			(show_name no)
@@
 			(project "engineering_plane"
 				(path "/f9a2ded0-d803-4be9-b2f5-4dda0f6b4d9a/9c29d4f9-b687-4678-a7ec-dae4a703e307"
-					(reference "R28")
+					(reference "R25")
 					(unit 1)
 				)
@@
 		(dnp no)
 		(fields_autoplaced yes)
-		(property "Reference" "#PWR080"
+		(property "Reference" "#PWR072"
 			(at 85.09 63.5 0)
 			(hide yes)
@@
 			(project "engineering_plane"
 				(path "/f9a2ded0-d803-4be9-b2f5-4dda0f6b4d9a/9c29d4f9-b687-4678-a7ec-dae4a703e307"
-					(reference "#PWR080")
+					(reference "#PWR072")
 					(unit 1)
 				)
@@
 		(in_pos_files yes)
 		(dnp no)
-		(property "Reference" "C33"
+		(property "Reference" "C19"
 			(at 69.342 83.566 0)
 			(show_name no)
@@
 			(project "engineering_plane"
 				(path "/f9a2ded0-d803-4be9-b2f5-4dda0f6b4d9a/9c29d4f9-b687-4678-a7ec-dae4a703e307"
-					(reference "C33")
+					(reference "C19")
 					(unit 1)
 				)
@@
 		(dnp no)
 		(fields_autoplaced yes)
-		(property "Reference" "#PWR086"
+		(property "Reference" "#PWR078"
 			(at 147.32 64.77 0)
 			(hide yes)
@@
 			(project "engineering_plane"
 				(path "/f9a2ded0-d803-4be9-b2f5-4dda0f6b4d9a/9c29d4f9-b687-4678-a7ec-dae4a703e307"
-					(reference "#PWR086")
+					(reference "#PWR078")
 					(unit 1)
 				)
@@
 		(dnp no)
 		(fields_autoplaced yes)
-		(property "Reference" "R27"
+		(property "Reference" "R24"
 			(at 92.71 62.2299 90)
 			(show_name no)
@@
 			(project "engineering_plane"
 				(path "/f9a2ded0-d803-4be9-b2f5-4dda0f6b4d9a/9c29d4f9-b687-4678-a7ec-dae4a703e307"
-					(reference "R27")
+					(reference "R24")
 					(unit 1)
 				)
@@
 		(dnp no)
 		(fields_autoplaced yes)
-		(property "Reference" "R31"
+		(property "Reference" "R27"
 			(at 149.86 64.7699 90)
 			(show_name no)
@@
 			(project "engineering_plane"
 				(path "/f9a2ded0-d803-4be9-b2f5-4dda0f6b4d9a/9c29d4f9-b687-4678-a7ec-dae4a703e307"
-					(reference "R31")
+					(reference "R27")
 					(unit 1)
 				)
@@
 		(dnp no)
 		(fields_autoplaced yes)
-		(property "Reference" "#PWR085"
+		(property "Reference" "#PWR077"
 			(at 151.13 72.39 0)
 			(hide yes)
@@
 			(project "engineering_plane"
 				(path "/f9a2ded0-d803-4be9-b2f5-4dda0f6b4d9a/9c29d4f9-b687-4678-a7ec-dae4a703e307"
-					(reference "#PWR085")
+					(reference "#PWR077")
 					(unit 1)
 				)
@@
 		(dnp no)
 		(fields_autoplaced yes)
-		(property "Reference" "R25"
+		(property "Reference" "R22"
 			(at 87.63 63.4999 90)
 			(show_name no)
@@
 			(project "engineering_plane"
 				(path "/f9a2ded0-d803-4be9-b2f5-4dda0f6b4d9a/9c29d4f9-b687-4678-a7ec-dae4a703e307"
-					(reference "R25")
+					(reference "R22")
 					(unit 1)
 				)
@@
 		(dnp no)
 		(fields_autoplaced yes)
-		(property "Reference" "R30"
+		(property "Reference" "R26"
 			(at 100.33 60.9599 90)
 			(show_name no)
@@
 			(project "engineering_plane"
 				(path "/f9a2ded0-d803-4be9-b2f5-4dda0f6b4d9a/9c29d4f9-b687-4678-a7ec-dae4a703e307"
-					(reference "R30")
+					(reference "R26")
 					(unit 1)
 				)
@@
 		(dnp no)
 		(fields_autoplaced yes)
-		(property "Reference" "#PWR084"
+		(property "Reference" "#PWR076"
 			(at 95.25 82.55 0)
 			(hide yes)
@@
 			(project "engineering_plane"
 				(path "/f9a2ded0-d803-4be9-b2f5-4dda0f6b4d9a/9c29d4f9-b687-4678-a7ec-dae4a703e307"
-					(reference "#PWR084")
+					(reference "#PWR076")
 					(unit 1)
 				)
@@
 		(dnp no)
 		(fields_autoplaced yes)
-		(property "Reference" "#PWR079"
+		(property "Reference" "#PWR071"
 			(at 66.04 91.44 0)
 			(hide yes)
@@
 			(project "engineering_plane"
 				(path "/f9a2ded0-d803-4be9-b2f5-4dda0f6b4d9a/9c29d4f9-b687-4678-a7ec-dae4a703e307"
-					(reference "#PWR079")
+					(reference "#PWR071")
 					(unit 1)
 				)
@@
 		(dnp no)
 		(fields_autoplaced yes)
-		(property "Reference" "#PWR078"
+		(property "Reference" "#PWR070"
 			(at 53.34 80.01 0)
 			(hide yes)
@@
 			(project "engineering_plane"
 				(path "/f9a2ded0-d803-4be9-b2f5-4dda0f6b4d9a/9c29d4f9-b687-4678-a7ec-dae4a703e307"
-					(reference "#PWR078")
+					(reference "#PWR070")
 					(unit 1)
 				)
@@
 		(in_pos_files yes)
 		(dnp no)
-		(property "Reference" "#PWR082"
+		(property "Reference" "#PWR074"
 			(at 93.98 88.9 0)
 			(hide yes)
@@
 			(project "engineering_plane"
 				(path "/f9a2ded0-d803-4be9-b2f5-4dda0f6b4d9a/9c29d4f9-b687-4678-a7ec-dae4a703e307"
-					(reference "#PWR082")
+					(reference "#PWR074")
 					(unit 1)
 				)
@@
 		(dnp no)
 		(fields_autoplaced yes)
-		(property "Reference" "#PWR081"
+		(property "Reference" "#PWR073"
 			(at 90.17 62.23 0)
 			(hide yes)
@@
 			(project "engineering_plane"
 				(path "/f9a2ded0-d803-4be9-b2f5-4dda0f6b4d9a/9c29d4f9-b687-4678-a7ec-dae4a703e307"
-					(reference "#PWR081")
+					(reference "#PWR073")
 					(unit 1)
 				)
@@
 		(dnp no)
 		(fields_autoplaced yes)
-		(property "Reference" "#PWR087"
+		(property "Reference" "#PWR079"
 			(at 147.32 92.71 0)
 			(hide yes)
@@
 			(project "engineering_plane"
 				(path "/f9a2ded0-d803-4be9-b2f5-4dda0f6b4d9a/9c29d4f9-b687-4678-a7ec-dae4a703e307"
-					(reference "#PWR087")
+					(reference "#PWR079")
 					(unit 1)
 				)
@@
 		(dnp no)
 		(fields_autoplaced yes)
-		(property "Reference" "#PWR083"
+		(property "Reference" "#PWR075"
 			(at 97.79 60.96 0)
 			(hide yes)
@@
 			(project "engineering_plane"
 				(path "/f9a2ded0-d803-4be9-b2f5-4dda0f6b4d9a/9c29d4f9-b687-4678-a7ec-dae4a703e307"
-					(reference "#PWR083")
-					(unit 1)
-				)
+					(reference "#PWR075")
+					(unit 1)
+				)

Commit message: Revised componenents, need to route
Parts:
- removed C18: 22u, Capacitor_SMD:C_1206_3216Metric, symbol Device:C
- removed C19: 100n, Capacitor_SMD:C_0603_1608Metric, symbol Device:C
- removed R21, R23: 22, PCM_SparkFun-Resistor:R_0603_1608Metric, symbol PCM_SparkFun-Resistor:R
- removed R22, R24, R25, R26, R27: 10k, PCM_SparkFun-Resistor:R_0603_1608Metric, symbol PCM_SparkFun-Resistor:R
- added C601: 22uF, PCM_JLCPCB:C_1206, symbol PCM_JLCPCB-Capacitors:1206,22uF,(2)
- added C602: 100nF, PCM_JLCPCB:C_0402, symbol PCM_JLCPCB-Capacitors:0402,100nF,(2)
- added R601, R603: 22Ω, PCM_JLCPCB:R_0402, symbol PCM_JLCPCB-Resistors:0402,22Ω
- added R602, R604, R605, R606, R607: 10kΩ, PCM_JLCPCB:R_0402, symbol PCM_JLCPCB-Resistors:0402,10kΩ
- renumbered J15 to J601
Connections:
- net +3V3: now also C601.1, C602.1, R602.1, R604.1, R605.1, R606.1, R607.1
- net GND: now also C601.2, C602.2
- net sd_cs: now also R604.2
- net at J601.1 (DAT2): now also R606.2
- net at J601.3 (CMD): now also R601.2, R602.2
- net at J601.5 (CLK): now also R603.2
- net at J601.8 (DAT1): now also R607.2
- net sd_data renamed SPI4.MISO
- net SPI4.MISO: now also R605.2
- new net SPI4.MOSI: R601.1
- new net SPI4.SCLK: R603.1
