File: power.kicad_sch (KiCad schematic)
At the start: 22 parts, among them U1 TPS54302DDCR, U2 TPS54302DDCR

Commit message: feat: new inductor.exe
Parts:
- L2: footprint Inductor_SMD:L_7.3x7.3_H4.5 -> eng_plane_lib:7447714220
Changed lines of the file:
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@@
 			)
 		)
-		(property "Footprint" "Inductor_SMD:L_7.3x7.3_H4.5"
+		(property "Footprint" "eng_plane_lib:7447714220"
 			(at 234.95 90.17 0)
 			(hide yes)

Commit message: feat: final changes, sent to prod
Parts:
- added C24, C32: 0.1u, Capacitor_SMD:C_0603_1608Metric, symbol Device:C
- C27: renamed from C10; footprint Capacitor_SMD:C_0603_1608Metric -> Capacitor_SMD:C_0805_2012Metric
- renumbered C1 to C20, C2 to C21, C3 to C22, C5 to C23, C7 to C25, C8 to C26, C12 to C28, C13 to C29, C14 to C30, C17 to C31, C18 to C33, C19 to C34, C21 to C35, L1 to L4, L2 to L5, R5 to R28, R6 to R29, R15 to R30, R16 to R31, U1 to U2, U2 to U3
Connections:
- net +5V: now also C24.1
- net +6V: now also C32.2
- net GND: now also C24.2, C32.1
Other:
- moved on the sheet: C20, C21, C22, C23, C33, C34, C35, L4, R30, R31, U2

Commit message: Revised componenents, need to route
Parts:
- removed C20, C21, C28, C29: 10u, Capacitor_SMD:C_1206_3216Metric, symbol Device:C
- removed C22, C23, C24, C30, C31, C32: 0.1u, Capacitor_SMD:C_0603_1608Metric, symbol Device:C
- removed C25, C26, C33, C34: 22u, Capacitor_SMD:C_1206_3216Metric, symbol Device:C
- removed C27, C35: 100p, Capacitor_SMD:C_0805_2012Metric, symbol Device:C
- removed R28, R30: 100k, PCM_SparkFun-Resistor:R_0603_1608Metric, symbol PCM_SparkFun-Resistor:R
- removed R31: 11k, PCM_SparkFun-Resistor:R_0603_1608Metric, symbol PCM_SparkFun-Resistor:R
- added C701, C702, C711, C712: 10uF, PCM_JLCPCB:C_1206, symbol PCM_JLCPCB-Capacitors:1206,10uF
- added C703, C705, C707, C713, C715: 100nF, PCM_JLCPCB:C_0603, symbol PCM_JLCPCB-Capacitors:0603,100nF
- added C704, C706: 1uF, PCM_JLCPCB:C_0402, symbol PCM_JLCPCB-Capacitors:0402,1uF
- added C708, C709, C716, C717: 22uF, PCM_JLCPCB:C_1206, symbol PCM_JLCPCB-Capacitors:1206,22uF,(2)
- added C710, C718: 100pF, PCM_JLCPCB:C_0603, symbol PCM_JLCPCB-Capacitors:0603,100pF
- added C714: 100nF, PCM_JLCPCB:C_0402, symbol PCM_JLCPCB-Capacitors:0402,100nF,(2)
- added IC701: LP5907MFX-3.3_NOPB, eng_plane_lib:SOT95P280X145-5M, symbol eng_plane_lib:LP5907MFX-3.3_NOPB
- added R701, R703: 100kΩ, PCM_JLCPCB:R_0603, symbol PCM_JLCPCB-Resistors:0603,100kΩ
- added R704: 11kΩ, PCM_JLCPCB:R_0603, symbol PCM_JLCPCB-Resistors:0603,11kΩ
- renumbered L4 to L701, L5 to L702, R29 to R702, U2 to U701, U3 to U702
Connections:
- net +5V: now also C704.1, C707.1, C708.1, C709.1, C710.1, IC701.1 (IN), IC701.3 (EN), R701.1
- net +6V: now also C715.1, C716.1, C717.1, C718.1, R703.1
- net 5v_div: now also C710.2, R701.2
- net 6v_div: now also C718.2, R703.2, R704.1
- net GND: now also C701.2, C702.2, C703.2, C704.2, C706.2, C707.2, C708.2, C709.2, C711.2, C712.2, C713.2, C715.2, C716.2, C717.2, IC701.2 (GND), R704.2
- net VBATT: now also C701.1, C702.1, C703.1, C711.1, C712.1, C713.1
- net at U702.6 (BOOT): now also C714.1
- net at L702.1, U702.2 (SW): now also C714.2
- net at L701.1, U701.2 (SW): now also C705.2
- net at U701.6 (BOOT): now also C705.1
- new net +3V3: C706.1, IC701.5 (OUT)
Other:
- note added: "3V3 LDO"
- moved on the sheet: L701

Commit message: finished routing
Parts:
- added TP701, TP702, TP703: 1.0mm, PCM_SparkFun-Connector:TestPoint-1.0mm, symbol PCM_SparkFun-Connector:TestPoint_1.0mm
Connections:
- net +5V: now also TP701.1
- net +6V: now also TP702.1
- net GND: now also TP703.1
Other:
- note added: "Have to externally source, not on jlc"
