File: ESC.kicad_sch (KiCad schematic)
At the start: 3 parts, among them J1101 Conn_01x03

Commit message: rev2 additional thingis
Parts:
- removed J1101: Conn_01x03, eng_plane_lib:1718564003, symbol Connector_Generic:Conn_01x03
- added J1101: B3B-XH-A__LF__SN_, eng_plane_lib:JST_B3B-XH-A__LF__SN_, symbol eng_plane_lib:B3B-XH-A__LF__SN_
Connections:
- net GND: now also J1101.1
- net at R1101.1, R1102.1: now also J1101.3
